File: Hardware/RevA/KiCad/LoLSnakes.kicad_pcb (KiCad board)
At the start: 2 copper layers, 74.9 x 64.8 mm, 157 parts, among them J1 ARDUINO, SW1 Encoder

Commit message: updated buzzer footprint
Parts:
- BZ1: value Buzzer -> BUZZER; footprint LoLSnakes:buzzer_tmb -> LoLSnakes:buzzer
- turned BZ1 to 0 degrees
Routing:
- net Net-(BZ1-Pad2): track 15.6 -> 10.7 mm
- net Net-(BZ1-Pad1): track 63.8 -> 67.6 mm
Changed lines of the file:
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@@
 (kicad_pcb (version 4) (host pcbnew 4.0.7)
   (general
-    (links 289)
-    (no_connects 0)
+    (links 291)
+    (no_connects 1)
     (area 108.829499 78.349499 185.007017 144.780001)
     (thickness 1.6)
     (drawings 2)
-    (tracks 531)
+    (tracks 534)
     (zones 0)
     (modules 157)
@@
     (34 B.Paste user)
     (35 F.Paste user)
-    (36 B.SilkS user hide)
+    (36 B.SilkS user)
     (37 F.SilkS user)
     (38 B.Mask user)
@@
     )
   )
-  (module LoLSnakes:buzzer_tmb (layer B.Cu)
-    (at 118.745 134.62 90)
-    (descr "Buzzer, TMB")
-    (tags buzzer)
-    (autoplace_cost180 10)
-    (fp_text reference BZ1 (at 0 3.683 90) (layer B.SilkS)
-      (effects (font (size 0.99822 0.99822) (thickness 0.19812)) (justify mirror))
-    )
-    (fp_text value Buzzer (at 0 -3.556 90) (layer B.SilkS)
-      (effects (font (size 0.99822 0.99822) (thickness 0.19812)) (justify mirror))
-    )
-    (fp_circle (center 0 0) (end 2.794 0.127) (layer B.SilkS) (width 0.2))
-    (pad 2 thru_hole circle (at -3.8 0 90) (size 1.5 1.5) (drill 0.8) (layers *.Cu *.Mask B.SilkS)
-      (net 1 "Net-(BZ1-Pad2)"))
-    (pad 1 thru_hole circle (at 3.8 0 90) (size 1.5 1.5) (drill 0.8) (layers *.Cu *.Mask B.SilkS)
-      (net 2 "Net-(BZ1-Pad1)"))
-    (model ${KIPRJMOD}/3D-Models/buzzer_tmb.wrl
-      (at (xyz 0 0 0))
-      (scale (xyz 1 1 1))
-      (rotate (xyz 0 0 0))
-    )
-  )
   (module LoLSnakes:arduino_header_extended (layer F.Cu)
     (at 148.59 105.41)
@@
       (xy 3.92176 0.64516)) (layer B.SilkS) (width 0.00254))
   )
+  (module LoLSnakes:buzzer (layer B.Cu)
+    (at 118.745 134.62)
+    (descr Buzzer)
+    (tags buzzer)
+    (autoplace_cost180 10)
+    (fp_text reference BZ1 (at 0 0) (layer B.SilkS)
+      (effects (font (size 0.99822 0.99822) (thickness 0.19812)) (justify mirror))
+    )
+    (fp_text value BUZZER (at 0 5.969) (layer B.SilkS) hide
+      (effects (font (size 0.99822 0.99822) (thickness 0.19812)) (justify mirror))
+    )
+    (fp_circle (center 0 0) (end 5.08 1.27) (layer B.SilkS) (width 0.15))
+    (pad 1 thru_hole circle (at 0 -3.175) (size 2 2) (drill 1) (layers *.Cu *.Mask)
+      (net 2 "Net-(BZ1-Pad1)"))
+    (pad 2 thru_hole circle (at 0 3.175) (size 2 2) (drill 1) (layers *.Cu *.Mask)
+      (net 1 "Net-(BZ1-Pad2)"))
+    (pad 2 thru_hole circle (at -2.54 0) (size 2 2) (drill 1) (layers *.Cu *.Mask)
+      (net 1 "Net-(BZ1-Pad2)"))
+    (pad 1 thru_hole circle (at 2.54 0) (size 2 2) (drill 1) (layers *.Cu *.Mask)
+      (net 2 "Net-(BZ1-Pad1)"))
+    (model ${KIPRJMOD}/3D-Models/buzzer.wrl
+      (at (xyz 0 0 0))
+      (scale (xyz 1 1 1))
+      (rotate (xyz 0 0 0))
+    )
+  )
   (gr_text "LoLSnakes\nRevA" (at 115.57 98.425 90) (layer B.SilkS)
     (effects (font (size 1.5 1.5) (thickness 0.3)) (justify right mirror))
@@
     (effects (font (size 1.5 1.5) (thickness 0.3)) (justify left mirror))
   )
-  (segment (start 114.935 128.905) (end 111.76 125.73) (width 0.25) (layer F.Cu) (net 1))
-  (segment (start 114.935 134.61) (end 114.935 128.905) (width 0.25) (layer F.Cu) (net 1))
-  (segment (start 118.745 138.42) (end 114.935 134.61) (width 0.25) (layer F.Cu) (net 1))
-  (segment (start 118.745 130.82) (end 120.96004 130.82) (width 0.25) (layer F.Cu) (net 2))
-  (segment (start 120.96004 130.82) (end 125.79604 125.984) (width 0.25) (layer F.Cu) (net 2))
-  (segment (start 139.954 125.984) (end 175.514 125.984) (width 0.25) (layer F.Cu) (net 2))
+  (segment (start 111.76 125.73) (end 114.935 128.905) (width 0.25) (layer F.Cu) (net 1))
+  (segment (start 114.935 133.35) (end 116.205 134.62) (width 0.25) (layer F.Cu) (net 1))
+  (segment (start 114.935 132.715) (end 114.935 133.35) (width 0.25) (layer F.Cu) (net 1))
+  (segment (start 114.935 128.905) (end 114.935 132.715) (width 0.25) (layer F.Cu) (net 1))
+  (segment (start 121.285 134.62) (end 120.33504 133.67004) (width 0.25) (layer F.Cu) (net 2))
+  (segment (start 120.33504 133.67004) (end 120.33504 131.445) (width 0.25) (layer F.Cu) (net 2))
+  (segment (start 125.79604 125.984) (end 120.33504 131.445) (width 0.25) (layer F.Cu) (net 2))
+  (segment (start 179.07 129.54) (end 175.514 125.984) (width 0.25) (layer F.Cu) (net 2))
   (segment (start 125.79604 125.984) (end 139.954 125.984) (width 0.25) (layer F.Cu) (net 2))
-  (segment (start 175.514 125.984) (end 179.07 129.54) (width 0.25) (layer F.Cu) (net 2))
+  (segment (start 139.954 125.984) (end 175.514 125.984) (width 0.25) (layer F.Cu) (net 2))
+  (segment (start 120.33504 131.445) (end 118.745 131.445) (width 0.25) (layer F.Cu) (net 2))
   (segment (start 119.38 87.63) (end 120.278026 86.731974) (width 0.25) (layer F.Cu) (net 3))
   (segment (start 120.278026 86.731974) (end 124.088026 86.731974) (width 0.25) (layer F.Cu) (net 3))
